Commit message: [Update] fixes to mounts.py and urdf.xacro files

File: clearpath_mounts_description/urdf/boss_male.urdf.xacro (robot description, xacro)
@@ -1,5 +1,5 @@
 <?xml version="1.0"?>
 <robot xmlns:xacro="http://wiki.ros.org/xacro">
-  <xacro:macro name="boss_male" params="name parent_link *origin">
+  <xacro:macro name="boss_male" params="name parent_link model *origin">
     <xacro:if value="${model == 'UNC_58'}">
         <xacro:property name="mesh_x" value="0.030"/>
@@ -17,5 +17,5 @@
       <collision>
         <geometry>
-          <cylinder radius="${mesh_x}/2.0" length="${mesh_z}" />
+          <cylinder radius="${mesh_x/2.0}" length="${mesh_z}" />
         </geometry>
         <origin xyz="0 0 0" rpy="${pi/2} 0 0" />

Commit message: [Update] Add scale factor in urdfs importing .stl meshes

File: clearpath_mounts_description/urdf/boss_male.urdf.xacro (robot description, xacro)
@@ -6,5 +6,5 @@
         <xacro:property name="mesh_y" value="0.030"/>
         <xacro:property name="mesh_z" value="0.021"/>
-        <xacro:property name="mesh" value="package://clearpath_mounts_description/meshes/boss_male/137-0040-00.stl"/>
+        <xacro:property name="mesh" value="package://clearpath_mounts_description/meshes/boss_male/137-0040-00.stl" scale="0.001 0.001 0.001"/>
     </xacro:if>
     <link name="${name}_link">

File: clearpath_platform_description/urdf/max/wheels/front_wheel.urdf.xacro (robot description, xacro)
@@ -11,5 +11,5 @@
         <origin xyz="0 0 0" rpy="0 0 0" />
         <geometry>
-          <mesh filename="package://clearpath_platform_description/meshes/max/front_wheel.stl" />
+          <mesh filename="package://clearpath_platform_description/meshes/max/front_wheel.stl" scale="0.001 0.001 0.001"/>
         </geometry>
       </visual>

File: clearpath_platform_description/urdf/max/wheels/rear_wheel.urdf.xacro (robot description, xacro)
@@ -11,5 +11,5 @@
         <origin xyz="0 0 0" rpy="0 0 0" />
         <geometry>
-          <mesh filename="package://clearpath_platform_description/meshes/max/rear_wheel.stl" />
+          <mesh filename="package://clearpath_platform_description/meshes/max/rear_wheel.stl" scale="0.001 0.001 0.001" />
         </geometry>
       </visual>

File: clearpath_sensors_description/urdf/ardusimple_RTKLite.urdf.xacro (robot description, xacro)
@@ -6,5 +6,5 @@
         <origin xyz="0 0 0" rpy="0 0 0" />
         <geometry>
-          <mesh filename="package://clearpath_sensors_description/meshes/136-0071-00.stl"/>
+          <mesh filename="package://clearpath_sensors_description/meshes/136-0071-00.stl" scale="0.001 0.001 0.001"/>
         </geometry>
         <material name="ardusimple_white">
@@ -15,5 +15,5 @@
         <origin xyz="0 0 0" rpy="0 0 0" />
         <geometry>
-          <mesh filename="package://clearpath_sensors_description/meshes/136-0071-00.stl"/>
+          <mesh filename="package://clearpath_sensors_description/meshes/136-0071-00.stl" scale="0.001 0.001 0.001"/>
         </geometry>
       </collision>

Commit message: [Update] Add scale factor in urdfs importing .stl meshes

File: clearpath_mounts_description/urdf/boss_male.urdf.xacro (robot description, xacro)
@@ -2,9 +2,10 @@
 <robot xmlns:xacro="http://wiki.ros.org/xacro">
   <xacro:macro name="boss_male" params="name parent_link model *origin">
+    <xacro:property name="mesh_scale" value="0.001 0.001 0.001"/>
     <xacro:if value="${model == 'UNC_58'}">
         <xacro:property name="mesh_x" value="0.030"/>
         <xacro:property name="mesh_y" value="0.030"/>
         <xacro:property name="mesh_z" value="0.021"/>
-        <xacro:property name="mesh" value="package://clearpath_mounts_description/meshes/boss_male/137-0040-00.stl" scale="0.001 0.001 0.001"/>
+        <xacro:property name="mesh" value="package://clearpath_mounts_description/meshes/boss_male/137-0040-00.stl" scale="${mesh_scale}"/>
     </xacro:if>
     <link name="${name}_link">

File: clearpath_platform_description/urdf/max/wheels/front_wheel.urdf.xacro (robot description, xacro)
@@ -2,4 +2,5 @@
 <robot xmlns:xacro="http://ros.org/wiki/xacro" name="front_wheel">
   <xacro:macro name="front_wheel" params="wheel_prefix *joint_pose">
+    <xacro:property name="mesh_scale" value="0.001 0.001 0.001"/>
     <link name="${wheel_prefix}_wheel">
       <inertial>
@@ -11,5 +12,5 @@
         <origin xyz="0 0 0" rpy="0 0 0" />
         <geometry>
-          <mesh filename="package://clearpath_platform_description/meshes/max/front_wheel.stl" scale="0.001 0.001 0.001"/>
+          <mesh filename="package://clearpath_platform_description/meshes/max/front_wheel.stl" scale="${mesh_scale}"/>
         </geometry>
       </visual>

File: clearpath_platform_description/urdf/max/wheels/rear_wheel.urdf.xacro (robot description, xacro)
@@ -2,4 +2,5 @@
 <robot xmlns:xacro="http://ros.org/wiki/xacro" name="rear_wheel">
   <xacro:macro name="rear_wheel" params="wheel_prefix *joint_pose">
+    <xacro:property name="mesh_scale" value="0.001 0.001 0.001"/>
     <link name="${wheel_prefix}_wheel">
       <inertial>
@@ -11,5 +12,5 @@
         <origin xyz="0 0 0" rpy="0 0 0" />
         <geometry>
-          <mesh filename="package://clearpath_platform_description/meshes/max/rear_wheel.stl" scale="0.001 0.001 0.001" />
+          <mesh filename="package://clearpath_platform_description/meshes/max/rear_wheel.stl" scale="${mesh_scale}" />
         </geometry>
       </visual>

File: clearpath_sensors_description/urdf/ardusimple_RTKLite.urdf.xacro (robot description, xacro)
@@ -2,9 +2,10 @@
 <robot xmlns:xacro="http://www.ros.org/wiki/xacro">
   <xacro:macro name="ardusimple_RTKLite" params="name parent_link *origin">
+    <xacro:property name="mesh_scale" value="0.001 0.001 0.001"/>
     <link name="${name}_link">
       <visual>
         <origin xyz="0 0 0" rpy="0 0 0" />
         <geometry>
-          <mesh filename="package://clearpath_sensors_description/meshes/136-0071-00.stl" scale="0.001 0.001 0.001"/>
+          <mesh filename="package://clearpath_sensors_description/meshes/136-0071-00.stl" scale="${mesh_scale}"/>
         </geometry>
         <material name="ardusimple_white">
@@ -15,5 +16,5 @@
         <origin xyz="0 0 0" rpy="0 0 0" />
         <geometry>
-          <mesh filename="package://clearpath_sensors_description/meshes/136-0071-00.stl" scale="0.001 0.001 0.001"/>
+          <mesh filename="package://clearpath_sensors_description/meshes/136-0071-00.stl" scale="${mesh_scale}"/>
         </geometry>
       </collision>

Commit message: [Update] correct syntax in boss_male.urdf.xacro

File: clearpath_mounts_description/urdf/boss_male.urdf.xacro (robot description, xacro)
@@ -7,10 +7,10 @@
         <xacro:property name="mesh_y" value="0.030"/>
         <xacro:property name="mesh_z" value="0.021"/>
-        <xacro:property name="mesh" value="package://clearpath_mounts_description/meshes/boss_male/137-0040-00.stl" scale="${mesh_scale}"/>
+        <xacro:property name="mesh_filename" value="package://clearpath_mounts_description/meshes/boss_male/137-0040-00.stl"/>
     </xacro:if>
     <link name="${name}_link">
       <visual>
         <geometry>
-          <mesh filename="${mesh}" />
+          <mesh filename="${mesh_filename}" scale="${mesh_scale}"/>
         </geometry>
         <origin xyz="0 0 0" rpy="0 0 ${pi/2}" />

Commit message: [Updixes to urdf files

File: clearpath_mounts_description/urdf/boss_male.urdf.xacro (robot description, xacro)
@@ -14,5 +14,5 @@
           <mesh filename="${mesh_filename}" scale="${mesh_scale}"/>
         </geometry>
-        <origin xyz="0 0 0" rpy="0 0 ${pi/2}" />
+        <origin xyz="0 0 0" rpy="${M_PI/2} ${-M_PI/2} 0" />
       </visual>
       <collision>
@@ -20,5 +20,5 @@
           <cylinder radius="${mesh_x/2.0}" length="${mesh_z}" />
         </geometry>
-        <origin xyz="0 0 0" rpy="${pi/2} 0 0" />
+        <origin xyz="0 0 0" rpy="${M_PI/2} 0 0" />
       </collision>
     </link>

File: clearpath_platform_description/urdf/max/max.urdf.xacro (robot description, xacro)
@@ -19,5 +19,5 @@
     <!-- Max wheel macros -->
     <xacro:front_wheel wheel_prefix="front_left">
-      <origin xyz="${wheelbase} ${front_track/2} ${wheel_vertical_offset}" rpy="0 0 0" />
+      <origin xyz="${wheelbase} ${front_track/2} ${wheel_vertical_offset}" rpy="0 0 ${M_PI}" />
     </xacro:front_wheel>
     <xacro:front_wheel wheel_prefix="front_right">
@@ -28,10 +28,19 @@
     </xacro:rear_wheel>
     <xacro:rear_wheel wheel_prefix="rear_right">
-      <origin xyz="0 ${-rear_track/2} ${wheel_vertical_offset}" rpy="0 0 0" />
+      <origin xyz="0 ${-rear_track/2} ${wheel_vertical_offset}" rpy="0 0 ${M_PI}" />
     </xacro:rear_wheel>
+    <!-- Base footprint is on the mid-plane of the vehicle coincident with the rear axis plane and the ground plane-->
+    <link name="base_footprint">
+      <visual>
+        <origin xyz="0 0 0" rpy="0 0 0" />
+        <geometry>
+          <sphere radius="0.05"/>
+        </geometry>
+      </visual>
+    </link>
     <!-- Base link is on the mid-plane of the vehicle coincident with the rear axis -->
     <link name="base_link">
       <visual>
-        <origin xyz="0 0 0.325" rpy="0 0 0" />
+        <origin xyz="0 0 0" rpy="0 0 0" />
         <geometry>
           <sphere radius="0.1"/>
@@ -39,4 +48,9 @@
       </visual>
     </link>
+    <joint name="base_link_joint" type="fixed">
+      <origin xyz="0 0 0.335" rpy="0 0 0"/>
+      <parent link="base_footprint"/>
+      <child link="base_link"/>
+    </joint>
   </xacro:macro>
 </robot>

File: clearpath_platform_description/urdf/max/wheels/front_wheel.urdf.xacro (robot description, xacro)
@@ -10,7 +10,7 @@
       </inertial>
       <visual>
-        <origin xyz="0 0 0" rpy="0 0 0" />
+        <origin xyz="0 0 0" rpy="${M_PI/2} 0 0" />
         <geometry>
-          <mesh filename="package://clearpath_platform_description/meshes/max/front_wheel.stl" scale="${mesh_scale}"/>
+          <mesh filename="package://clearpath_platform_description/meshes/max/max_front_wheel.stl" scale="${mesh_scale}"/>
         </geometry>
       </visual>

File: clearpath_platform_description/urdf/max/wheels/rear_wheel.urdf.xacro (robot description, xacro)
@@ -10,7 +10,7 @@
       </inertial>
       <visual>
-        <origin xyz="0 0 0" rpy="0 0 0" />
+        <origin xyz="0 0 0" rpy="0 0 ${M_PI/2}" />
         <geometry>
-          <mesh filename="package://clearpath_platform_description/meshes/max/rear_wheel.stl" scale="${mesh_scale}" />
+          <mesh filename="package://clearpath_platform_description/meshes/max/max_rear_wheel.stl" scale="${mesh_scale}" />
         </geometry>
       </visual>
